File: Driver_Schem.kicad_sch (KiCad schematic)
At the start: 15 parts, among them J1 YO0221500000G, J2 YO0221500000G, U2 DRV8870DDA

Commit message: Add files via upload
New changes to the PCB
Parts:
- added J5, J7, J8, J9: Conn_01x01_Pin, symbol Connector:Conn_01x01_Pin
- added J6: Conn_01x05_Pin, symbol Connector:Conn_01x05_Pin
- added R10, R7, R8, R9: 0, symbol Device:R_Small_US
- U1: footprint (none) -> PGA460:PW16_TEX
Connections:
- net IO: now also J6.5 (Pin_5)
- net IOREG: now also U2.4 (VREF)
- net RXD: now also J6.2 (Pin_2)
- net TXD: now also J6.3 (Pin_3)
- net VPWR: now also J6.1 (Pin_1)
- net VX: now also J6.4 (Pin_4)
- net at R2.2, R4.1: now also J9.1 (Pin_1), R10.1, R8.2; no longer U1.7 (OUTB), U2.2 (IN2)
- net at R1.2, R3.1: now also J8.1 (Pin_1), R7.2, R9.1; no longer U1.5 (OUTA), U2.3 (IN1)
- new net: R7.1, U1.5 (OUTA)
- new net: R8.1, U1.7 (OUTB)
- new net: J7.1 (Pin_1), R10.2, U2.2 (IN2)
- new net: J5.1 (Pin_1), R9.2, U2.3 (IN1)
Other:
- note added: "From TI's App Note about this configuration: A limitation of the DRV8870 based solution is that the DRV8870 enters sleep mode when inactive. When the IN1 and IN2 pins are both low for approximately 1 ms, the DRV8870 device enters a low-power sleep mode where the outputs remain High-Z, and the devices uses micro-amperes of current. If the DRV8870 is powered up while both inputs are low, it immedia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"
- moved on the sheet: J1, R1, R2, R3, R4, R5, U2

Commit message: Add files via upload
This is the current PCB design. I am open to suggestions for changes.
Parts:
- removed R10, R7, R8, R9: 0, symbol Device:R_Small_US
- C1, C2, C3, C4, C5: footprint (none) -> Capacitor_SMD:C_0805_2012Metric
- J1, J2: footprint footprints:CONN_YO0221500000G_AMP -> YO0221500000G:CONN_YO0221500000G_AMP
- J5, J7, J8, J9: footprint (none) -> Connector_PinHeader_2.54mm:PinHeader_1x01_P2.54mm_Vertical
- J6: footprint (none) -> Connector_PinHeader_2.54mm:PinHeader_1x05_P2.54mm_Vertical
- R1, R2: value 33.2k -> 4.7k; footprint (none) -> Resistor_SMD:R_0805_2012Metric
- R3, R4: value 2.7k -> 0; footprint (none) -> Resistor_SMD:R_0805_2012Metric
- R5, R6: footprint (none) -> Resistor_SMD:R_0805_2012Metric
Connections:
- net GND: no longer R3.2, R4.2
- net IOREG: now also R1.1, R2.1
- net VX: no longer R1.1, R2.1
- net at J9.1 (Pin_1), R2.2, R4.1: now also U1.7 (OUTB)
- net at J8.1 (Pin_1), R1.2, R3.1: now also U1.5 (OUTA)
- net at J7.1 (Pin_1), U2.2 (IN2): now also R4.2
- net at J5.1 (Pin_1), U2.3 (IN1): now also R3.2
Other:
- note added: "PGA460"
- moved on the sheet: J5

Commit message: Add files via upload
This will be the most up to date PCB. Throw the 3D viewer on and rotate it for an easter egg.
Parts:
- removed R3, R4: 0, Resistor_SMD:R_0805_2012Metric, symbol Device:R_Small_US
- added R10, R7, R8, R9: 0, Resistor_SMD:R_0805_2012Metric, symbol Device:R_Small_US
- J1, J2: footprint YO0221500000G:CONN_YO0221500000G_AMP -> footprints:CONN_YO0221500000G_AMP
Connections:
- net at J9.1 (Pin_1), R2.2: now also R10.1, R8.2; no longer U1.7 (OUTB)
- net at J7.1 (Pin_1), U2.2 (IN2): now also R10.2
- net at J8.1 (Pin_1), R1.2: now also R7.2, R9.1; no longer U1.5 (OUTA)
- net at J5.1 (Pin_1), U2.3 (IN1): now also R9.2
- new net: R7.1, U1.5 (OUTA)
- new net: R8.1, U1.7 (OUTB)
Other:
- note removed: "PGA460"
- moved on the sheet: J5
