File: Power_Schem.kicad_sch (KiCad schematic)
At the start: 16 parts, among them U3 LMR33640ADDA

Commit message: Add files via upload
New changes to the PCB
Parts:
- renumbered Cboot to Cboot2, Cin to Cin3, Cinx to Cinx1, Cout to Cout3, Coutx to Coutx1, Cvcc to Cvcc1, Rfbt to Rfbt2, Rpg to Rpg1
Connections:
- net 5V_Out renamed 5V_FPGA_Power
Changed lines of the file:
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@@
 		)
 	)
-	(label "5V_Out"
+	(hierarchical_label "V_Battery"
+		(shape input)
+		(at 54.61 62.23 180)
+		(effects
+			(font
+				(size 1.27 1.27)
+			)
+			(justify right)
+		)
+	)
+	(hierarchical_label "5V_FPGA_Power"
+		(shape input)
 		(at 259.08 64.77 0)
 		(effects
@@
 				(size 1.27 1.27)
 			)
-			(justify left bottom)
-		)
-	)
-	(label "V_Battery"
-		(at 54.61 62.23 0)
-		(effects
-			(font
-				(size 1.27 1.27)
-			)
-			(justify left bottom)
+			(justify left)
 		)
 	)
@@
 		(on_board yes)
 		(dnp no)
-		(property "Reference" "Cboot"
+		(property "Reference" "Cboot2"
 			(at 161.798 55.499 0)
 			(effects
@@
 			(project ""
 				(path "/f02116dc-3d6e-45e4-b4ab-5ea900e13651/307a8eb5-3be3-461a-96d2-9ca06d1bde49"
-					(reference "Cboot")
+					(reference "Cboot2")
 					(unit 1)
 				)
@@
 		(on_board yes)
 		(dnp no)
-		(property "Reference" "Rfbt"
+		(property "Reference" "Rfbt2"
 			(at 199.39 70.358 0)
 			(effects
@@
 			(project "FPGA_Anemometer_PCB"
 				(path "/f02116dc-3d6e-45e4-b4ab-5ea900e13651/307a8eb5-3be3-461a-96d2-9ca06d1bde49"
-					(reference "Rfbt")
+					(reference "Rfbt2")
 					(unit 1)
 				)
@@
 		(dnp no)
 		(fields_autoplaced yes)
-		(property "Reference" "Cinx"
+		(property "Reference" "Cinx1"
 			(at 113.03 73.6662 0)
 			(effects
@@
 			(project ""
 				(path "/f02116dc-3d6e-45e4-b4ab-5ea900e13651/307a8eb5-3be3-461a-96d2-9ca06d1bde49"
-					(reference "Cinx")
+					(reference "Cinx1")
 					(unit 1)
 				)
@@
 		(dnp no)
 		(fields_autoplaced yes)
-		(property "Reference" "Cin"
+		(property "Reference" "Cin3"
 			(at 99.06 73.6662 0)
 			(effects
@@
 			(project "FPGA_Anemometer_PCB"
 				(path "/f02116dc-3d6e-45e4-b4ab-5ea900e13651/307a8eb5-3be3-461a-96d2-9ca06d1bde49"
-					(reference "Cin")
+					(reference "Cin3")
 					(unit 1)
 				)
@@
 		(dnp no)
 		(fields_autoplaced yes)
-		(property "Reference" "Coutx"
+		(property "Reference" "Coutx1"
 			(at 210.82 74.9362 0)
 			(effects
@@
 			(project "FPGA_Anemometer_PCB"
 				(path "/f02116dc-3d6e-45e4-b4ab-5ea900e13651/307a8eb5-3be3-461a-96d2-9ca06d1bde49"
-					(reference "Coutx")
+					(reference "Coutx1")
 					(unit 1)
 				)
@@
 		(dnp no)
 		(fields_autoplaced yes)
-		(property "Reference" "Cout"
+		(property "Reference" "Cout3"
 			(at 224.79 74.9362 0)
 			(effects
@@
 			(project "FPGA_Anemometer_PCB"
 				(path "/f02116dc-3d6e-45e4-b4ab-5ea900e13651/307a8eb5-3be3-461a-96d2-9ca06d1bde49"
-					(reference "Cout")
+					(reference "Cout3")
 					(unit 1)
 				)
@@
 		(on_board yes)
 		(dnp no)
-		(property "Reference" "Rpg"
+		(property "Reference" "Rpg1"
 			(at 162.306 74.803 90)
 			(effects
@@
 			(project ""
 				(path "/f02116dc-3d6e-45e4-b4ab-5ea900e13651/307a8eb5-3be3-461a-96d2-9ca06d1bde49"
-					(reference "Rpg")
+					(reference "Rpg1")
 					(unit 1)
 				)
@@
 		(dnp no)
 		(fields_autoplaced yes)
-		(property "Reference" "Cvcc"
+		(property "Reference" "Cvcc1"
 			(at 127 78.7462 0)
 			(effects
@@
 			(project ""
 				(path "/f02116dc-3d6e-45e4-b4ab-5ea900e13651/307a8eb5-3be3-461a-96d2-9ca06d1bde49"
-					(reference "Cvcc")
-					(unit 1)
-				)
+					(reference "Cvcc1")
+					(unit 1)
+				)

Commit message: Add files via upload
This is the current PCB design. I am open to suggestions for changes.
Parts:
- Cboot2, Cin1, Cin2, Cin3, Cinx1, Cout1, Cout2, Cout3, Coutx1, Cvcc1: footprint (none) -> Capacitor_SMD:C_0805_2012Metric
- Cff1: renamed from Cboot1; footprint (none) -> Capacitor_SMD:C_0805_2012Metric
- L1: footprint (none) -> SRP1038A-150M:IND_SRP1038A_BRN
- Rfbt1, Rfbt2, Rpg1: footprint (none) -> Resistor_SMD:R_0805_2012Metric
Connections:
- net BOOT: now reaches Cboot2.1, U3.7 (BOOT)
- net SW: now reaches Cboot2.2, L1.1, U3.8 (SW)
- net FB: now reaches Cff1.2, Rfbt1.2, Rfbt2.1, U3.5 (FB)
- net PG: now reaches Rpg1.1, U3.4 (PG)
- net VCC: now reaches Cvcc1.1, U3.6 (VCC)
Changed lines of the file:
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@@
+		)
+	)
+	(label "FB"
+		(at 161.29 69.85 0)
+		(effects
+			(font
+				(size 1.27 1.27)
+			)
+			(justify left bottom)
+		)
+	)
+	(label "SW"
+		(at 156.21 64.77 0)
+		(effects
+			(font
+				(size 1.27 1.27)
+			)
+			(justify left bottom)
+		)
+	)
+	(label "BOOT"
+		(at 152.4 53.34 0)
+		(effects
+			(font
+				(size 1.27 1.27)
+			)
+			(justify left bottom)
+		)
+	)
+	(label "PG"
+		(at 153.67 72.39 0)
+		(effects
+			(font
+				(size 1.27 1.27)
+			)
+			(justify left bottom)
+		)
+	)
+	(label "VCC"
+		(at 124.46 72.39 0)
+		(effects
+			(font
+				(size 1.27 1.27)
+			)
+			(justify left bottom)
 		)
 	)
@@
 			)
 		)
-		(property "Footprint" ""
+		(property "Footprint" "Capacitor_SMD:C_0805_2012Metric"
 			(at 160.02 57.15 0)
 			(effects
@@
 		(on_board yes)
 		(dnp no)
-		(property "Reference" "Cboot1"
+		(property "Reference" "Cff1"
 			(at 184.658 70.739 0)
 			(effects
@@
 			)
 		)
-		(property "Footprint" ""
+		(property "Footprint" "Capacitor_SMD:C_0805_2012Metric"
 			(at 182.88 72.39 0)
 			(effects
@@
 			(project "FPGA_Anemometer_PCB"
 				(path "/f02116dc-3d6e-45e4-b4ab-5ea900e13651/307a8eb5-3be3-461a-96d2-9ca06d1bde49"
-					(reference "Cboot1")
+					(reference "Cff1")
 					(unit 1)
 				)
@@
 			)
 		)
-		(property "Footprint" ""
+		(property "Footprint" "Capacitor_SMD:C_0805_2012Metric"
 			(at 71.12 74.93 0)
 			(effects
@@
 			)
 		)
-		(property "Footprint" ""
+		(property "Footprint" "Resistor_SMD:R_0805_2012Metric"
 			(at 195.58 81.28 0)
 			(effects
@@
 			)
 		)
-		(property "Footprint" ""
+		(property "Footprint" "Resistor_SMD:R_0805_2012Metric"
 			(at 195.58 71.12 0)
 			(effects
@@
 			)
 		)
-		(property "Footprint" ""
+		(property "Footprint" "Capacitor_SMD:C_0805_2012Metric"
 			(at 110.49 74.93 0)
 			(effects
@@
 			)
 		)
-		(property "Footprint" ""
+		(property "Footprint" "Capacitor_SMD:C_0805_2012Metric"
 			(at 96.52 74.93 0)
 			(effects
@@
 			)
 		)
-		(property "Footprint" ""
+		(property "Footprint" "Capacitor_SMD:C_0805_2012Metric"
 			(at 208.28 76.2 0)
 			(effects
@@
 			)
 		)
-		(property "Footprint" ""
+		(property "Footprint" "Capacitor_SMD:C_0805_2012Metric"
 			(at 247.65 76.2 0)
 			(effects
@@
 			)
 		)
-		(property "Footprint" ""
+		(property "Footprint" "Capacitor_SMD:C_0805_2012Metric"
 			(at 222.25 76.2 0)
 			(effects
@@
 			)
 		)
-		(property "Footprint" ""
+		(property "Footprint" "Resistor_SMD:R_0805_2012Metric"
 			(at 162.56 72.39 0)
 			(effects
@@
 			)
 		)
-		(property "Footprint" ""
+		(property "Footprint" "Capacitor_SMD:C_0805_2012Metric"
 			(at 124.46 80.01 0)
 			(effects
@@
 			)
 		)
-		(property "Footprint" ""
+		(property "Footprint" "Capacitor_SMD:C_0805_2012Metric"
 			(at 234.95 76.2 0)
 			(effects
@@
 			)
 		)
-		(property "Footprint" ""
+		(property "Footprint" "Capacitor_SMD:C_0805_2012Metric"
 			(at 83.82 74.93 0)
 			(effects
@@
 			)
 		)
-		(property "Footprint" ""
+		(property "Footprint" "SRP1038A-150M:IND_SRP1038A_BRN"
 			(at 171.45 64.77 0)
 			(effects

Commit message: Add files via upload
This will be the most up to date PCB. Throw the 3D viewer on and rotate it for an easter egg.
Parts:
- Cout1, Cout2, Cout3: footprint Capacitor_SMD:C_0805_2012Metric -> Capacitor_THT:CP_Radial_D8.0mm_P5.00mm
- L1: footprint SRP1038A-150M:IND_SRP1038A_BRN -> (none)
Connections:
- net BOOT: no longer names the net of Cboot2.1, U3.7 (BOOT)
- net FB: no longer names the net of Cff1.2, Rfbt1.2, Rfbt2.1, U3.5 (FB)
- net PG: no longer names the net of Rpg1.1, U3.4 (PG)
- net SW: no longer names the net of Cboot2.2, L1.1, U3.8 (SW)
- net VCC: no longer names the net of Cvcc1.1, U3.6 (VCC)
Changed lines of the file:
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@@
-		)
-	)
-	(label "FB"
-		(at 161.29 69.85 0)
-		(effects
-			(font
-				(size 1.27 1.27)
-			)
-			(justify left bottom)
-		)
-	)
-	(label "SW"
-		(at 156.21 64.77 0)
-		(effects
-			(font
-				(size 1.27 1.27)
-			)
-			(justify left bottom)
-		)
-	)
-	(label "BOOT"
-		(at 152.4 53.34 0)
-		(effects
-			(font
-				(size 1.27 1.27)
-			)
-			(justify left bottom)
-		)
-	)
-	(label "PG"
-		(at 153.67 72.39 0)
-		(effects
-			(font
-				(size 1.27 1.27)
-			)
-			(justify left bottom)
-		)
-	)
-	(label "VCC"
-		(at 124.46 72.39 0)
-		(effects
-			(font
-				(size 1.27 1.27)
-			)
-			(justify left bottom)
 		)
 	)
@@
 			)
 		)
-		(property "Footprint" "Capacitor_SMD:C_0805_2012Metric"
+		(property "Footprint" "Capacitor_THT:CP_Radial_D8.0mm_P5.00mm"
 			(at 247.65 76.2 0)
 			(effects
@@
 			)
 		)
-		(property "Footprint" "Capacitor_SMD:C_0805_2012Metric"
+		(property "Footprint" "Capacitor_THT:CP_Radial_D8.0mm_P5.00mm"
 			(at 222.25 76.2 0)
 			(effects
@@
 			)
 		)
-		(property "Footprint" "Capacitor_SMD:C_0805_2012Metric"
+		(property "Footprint" "Capacitor_THT:CP_Radial_D8.0mm_P5.00mm"
 			(at 234.95 76.2 0)
 			(effects
@@
 			)
 		)
-		(property "Footprint" "SRP1038A-150M:IND_SRP1038A_BRN"
+		(property "Footprint" ""
 			(at 171.45 64.77 0)
 			(effects
