File: FPGA_Anemometer_PCB/Driver_Schem.kicad_sch (KiCad schematic)
At the start: 22 parts, among them J1 YO0221500000G, J2 YO0221500000G, J5 Conn_01x01_Pin, J6 Conn_01x05_Pin, J7 Conn_01x01_Pin, J8 Conn_01x01_Pin, J9 Conn_01x01_Pin, U2 DRV8870DDA

Commit message: updated pcb
Parts:
- removed R10, R7, R8, R9: 0, Resistor_SMD:R_0805_2012Metric, symbol Device:R_Small_US
- added R3, R4: 0, Resistor_SMD:R_0805_2012Metric, symbol Device:R_Small_US
- J1, J2: footprint footprints:CONN_YO0221500000G_AMP -> YO0221500000G:CONN_YO0221500000G_AMP
Connections:
- net at J9.1 (Pin_1), R2.2: now also U1.7 (OUTB), R4.1
- net at J8.1 (Pin_1), R1.2: now also U1.5 (OUTA), R3.2
- net at J7.1 (Pin_1), U2.2 (IN2): now also R4.2
- net at J5.1 (Pin_1), U2.3 (IN1): now also R3.1
Other:
- note added: "PGA460"
- moved on the sheet: J5, U2
