File: FPGA_Anemometer_PCB/Power_Schem.kicad_sch (KiCad schematic)
At the start: 16 parts, among them U3 LMR33640ADDA

Commit message: updated pcb
Parts:
- added R7: 0, Resistor_SMD:R_0805_2012Metric, symbol Device:R_Small_US
- Cout1, Cout2, Cout3: footprint Capacitor_THT:CP_Radial_D8.0mm_P5.00mm -> Capacitor_SMD:C_0805_2012Metric
- L1: footprint (none) -> SRP1038A-150M:IND_SRP1038A_BRN
Connections:
- net 5V_FPGA_Power: now also R7.2; no longer Cff1.1, Cout1.1, Cout2.1, Cout3.1, Coutx1.1, L1.2, Rfbt2.2, Rpg1.2
- net BOOT: now reaches Cboot2.1, U3.7 (BOOT)
- net SW: now reaches Cboot2.2, L1.1, U3.8 (SW)
- net FB: now reaches Cff1.2, Rfbt1.2, Rfbt2.1, U3.5 (FB)
- net PG: now reaches Rpg1.1, U3.4 (PG)
- net VCC: now reaches Cvcc1.1, U3.6 (VCC)
- new net: Cff1.1, Cout1.1, Cout2.1, Cout3.1, Coutx1.1, L1.2, R7.1, Rfbt2.2, Rpg1.2
Changed lines of the file:
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@@
+	(wire
+		(pts
+			(xy 256.54 64.77) (xy 259.08 64.77)
+		)
+		(stroke
+			(width 0)
+			(type default)
+		)
+	)
 	(wire
 		(pts
@@
 	(wire
 		(pts
-			(xy 247.65 64.77) (xy 259.08 64.77)
+			(xy 247.65 64.77) (xy 251.46 64.77)
 		)
 		(stroke
@@
 			(width 0)
 			(type default)
+		)
+	)
+	(label "FB"
+		(at 161.29 69.85 0)
+		(effects
+			(font
+				(size 1.27 1.27)
+			)
+			(justify left bottom)
+		)
+	)
+	(label "SW"
+		(at 156.21 64.77 0)
+		(effects
+			(font
+				(size 1.27 1.27)
+			)
+			(justify left bottom)
+		)
+	)
+	(label "BOOT"
+		(at 152.4 53.34 0)
+		(effects
+			(font
+				(size 1.27 1.27)
+			)
+			(justify left bottom)
+		)
+	)
+	(label "PG"
+		(at 153.67 72.39 0)
+		(effects
+			(font
+				(size 1.27 1.27)
+			)
+			(justify left bottom)
+		)
+	)
+	(label "VCC"
+		(at 124.46 72.39 0)
+		(effects
+			(font
+				(size 1.27 1.27)
+			)
+			(justify left bottom)
 		)
 	)
@@
 	)
 	(symbol
+		(lib_id "Device:R_Small_US")
+		(at 254 64.77 90)
+		(unit 1)
+		(exclude_from_sim no)
+		(in_bom yes)
+		(on_board yes)
+		(dnp no)
+		(fields_autoplaced yes)
+		(property "Reference" "R7"
+			(at 254 58.42 90)
+			(effects
+				(font
+					(size 1.27 1.27)
+				)
+			)
+		)
+		(property "Value" "0"
+			(at 254 60.96 90)
+			(effects
+				(font
+					(size 1.27 1.27)
+				)
+			)
+		)
+		(property "Footprint" "Resistor_SMD:R_0805_2012Metric"
+			(at 254 64.77 0)
+			(effects
+				(font
+					(size 1.27 1.27)
+				)
+				(hide yes)
+			)
+		)
+		(property "Datasheet" "~"
+			(at 254 64.77 0)
+			(effects
+				(font
+					(size 1.27 1.27)
+				)
+				(hide yes)
+			)
+		)
+		(property "Description" "Resistor, small US symbol"
+			(at 254 64.77 0)
+			(effects
+				(font
+					(size 1.27 1.27)
+				)
+				(hide yes)
+			)
+		)
+		(pin "1"
+		)
+		(pin "2"
+		)
+		(instances
+			(project ""
+				(path "/f02116dc-3d6e-45e4-b4ab-5ea900e13651/307a8eb5-3be3-461a-96d2-9ca06d1bde49"
+					(reference "R7")
+					(unit 1)
+				)
+			)
+		)
+	)
+	(symbol
 		(lib_id "Device:C_Small")
 		(at 96.52 74.93 0)
@@
 			)
 		)
-		(property "Footprint" "Capacitor_THT:CP_Radial_D8.0mm_P5.00mm"
+		(property "Footprint" "Capacitor_SMD:C_0805_2012Metric"
 			(at 247.65 76.2 0)
 			(effects
@@
 			)
 		)
-		(property "Footprint" "Capacitor_THT:CP_Radial_D8.0mm_P5.00mm"
+		(property "Footprint" "Capacitor_SMD:C_0805_2012Metric"
 			(at 222.25 76.2 0)
 			(effects
@@
 			)
 		)
-		(property "Footprint" "Capacitor_THT:CP_Radial_D8.0mm_P5.00mm"
+		(property "Footprint" "Capacitor_SMD:C_0805_2012Metric"
 			(at 234.95 76.2 0)
 			(effects
@@
 			)
 		)
-		(property "Footprint" ""
+		(property "Footprint" "SRP1038A-150M:IND_SRP1038A_BRN"
 			(at 171.45 64.77 0)
 			(effects
